File: radioCR_AFE_v1/rf_afe_v1.kicad_pcb (KiCad board)
At the start: 2 copper layers, 148.2 x 28.9 mm, 42 parts, among them J1 Conn_Coaxial, J2 Conn_Coaxial, U1 PHA-13LN, U2 BSF108+, U3 PHA-13LN, U4 RBP188, U5 PSA8A+, U6 TCBT-6G+, U7 PAT-3, U8 PAT-3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

Commit message: updated C1 footprint, regen bom
Parts:
- C1: footprint Capacitor_SMD:C_0603_1608Metric -> Capacitor_SMD:C_0805_2012Metric
- moved CR1 0.81 mm to (94.0, 99.1)
- moved CR2 0.81 mm to (94.0, 97.2)
- moved C3 0.77 mm to (96.4, 98.8)
- moved L1 0.50 mm to (99.5, 99.7)
- moved C1 0.33 mm to (103.0, 99.7)
Routing:
- net Net-(J1-In): track 9.44 -> 8.53 mm
Other:
- board text added: "VM/MSV/JSM + G3RA Collab IITK, TIFR/CRL, OSU"
- board text removed: "VM/MSV/JSM + G3 Collab IITK, TIFR/CRL, OSU"
